File: Filmoid Card.kicad_pcb (KiCad board)
At the start: 2 copper layers, 36 x 52 mm, 37 parts, among them SW1 SW_Push, SW2 SW_Push, U1 DHT11, U2 Seeeduino Xiao rp2040

Commit message: Add files via upload
Routing:
- net /Plex3: track 41.5 -> 45.1 mm, vias 6 -> 8
- net /Plex1: track 58.9 -> 56.3 mm
- net /Plex4: track 40.7 -> 43.0 mm
- net /Plex2: track 34.9 -> 36.7 mm
- net +3.3V: track 59.8 -> 58.6 mm
- net /SCL: track 46.2 -> 47.1 mm, vias 1 -> 2
- net /DHT11 data: track 49.3 -> 49.9 mm, vias 1 -> 6
